Commit message: added control with problems

File: robot/ur10/ur10.urdf (robot description, URDF)
Before this commit: robot ur10, 11 links, 10 joints
Links:
- link base_link: geometry collision mesh filename=base.stl; visual mesh filename=base.dae
- link forearm_link: geometry collision mesh filename=forearm.stl; visual mesh filename=forearm.dae
- link shoulder_link: geometry collision mesh filename=shoulder.stl; visual mesh filename=shoulder.dae
- link upper_arm_link: geometry collision mesh filename=upperarm.stl; visual mesh filename=upperarm.dae
- link wrist_1_link: geometry collision mesh filename=wrist1.stl; visual mesh filename=wrist1.dae
- link wrist_2_link: geometry collision mesh filename=wrist2.stl; visual mesh filename=wrist2.dae
- link wrist_3_link: geometry collision mesh filename=wrist3.stl; visual mesh filename=wrist3.dae
